Commit message: correct gripper pose

File: urdf/ur5_robotiq_camera.xacro (robot description, xacro)
@@ -6,5 +6,5 @@
     <xacro:include filename="$(find robotiq_gripper)/urdf/robotiq_85_gripper.urdf.xacro" />
     <xacro:robotiq_85_gripper prefix="" parent="tool0" >
-    <origin xyz="0 0 0.004" rpy="0 ${-pi/2} ${pi}"/>
+    <origin xyz="0 0 0.004" rpy="0 ${-pi/2} ${pi/2}"/>
     </xacro:robotiq_85_gripper>
     <!-- Include Simulated Realsense camera xacro -->

File: urdf/ur5_robotiq_description.xacro (robot description, xacro)
@@ -6,5 +6,5 @@
     <xacro:include filename="$(find robotiq_gripper)/urdf/robotiq_85_gripper.urdf.xacro" />
     <xacro:robotiq_85_gripper prefix="" parent="tool0" >
-    <origin xyz="0 0 0.004" rpy="0 ${-pi/2} ${pi}"/>
+    <origin xyz="0 0 0.004" rpy="0 ${-pi/2} ${pi/2}"/>
     </xacro:robotiq_85_gripper>
 </robot>
