Commit message: control real robot and gripper

File: urdf/ur.urdf.xacro (robot description, xacro)
@@ -1,96 +1,144 @@
 <?xml version="1.0"?>
 <robot xmlns:xacro="http://wiki.ros.org/xacro" name="$(arg name)">
-  <!-- robot name parameter -->
-  <xacro:arg name="name" default="ur"/>
-  <xacro:include filename="$(find ur_description)/urdf/ur_macro.xacro"/>
-  <!-- ros2 control include -->
-  <xacro:include filename="$(find ur5_robot_gripper)/urdf/ur.ros2_control.xacro" />
-  <xacro:include filename="$(find ur_description)/urdf/inc/ur_transmissions.xacro" />
-  <!-- possible 'ur_type' values: ur3, ur3e, ur5, ur5e, ur7e, ur10, ur10e, ur12e, ur16e, ur15, ur20, ur30 -->
-  <!-- the default value should raise an error in case this was called without defining the type -->
-  <xacro:arg name="ur_type" default="urXe"/>
-  <!-- parameters -->
-  <xacro:arg name="tf_prefix" default="" />
-  <xacro:arg name="joint_limit_params" default="$(find ur_description)/config/$(arg ur_type)/joint_limits.yaml"/>
-  <xacro:arg name="kinematics_params" default="$(find ur_description)/config/$(arg ur_type)/default_kinematics.yaml"/>
-  <xacro:arg name="physical_params" default="$(find ur_description)/config/$(arg ur_type)/physical_parameters.yaml"/>
-  <xacro:arg name="visual_params" default="$(find ur_description)/config/$(arg ur_type)/visual_parameters.yaml"/>
-  <xacro:arg name="transmission_hw_interface" default=""/>
-  <xacro:arg name="safety_limits" default="false"/>
-  <xacro:arg name="safety_pos_margin" default="0.15"/>
-  <xacro:arg name="safety_k_position" default="20"/>
-  <!-- ros2_control related parameters -->
-  <xacro:arg name="headless_mode" default="false" />
-  <xacro:arg name="robot_ip" default="0.0.0.0" />
-  <xacro:arg name="script_filename" default=""/>
-  <xacro:arg name="output_recipe_filename" default=""/>
-  <xacro:arg name="input_recipe_filename" default=""/>
-  <xacro:arg name="reverse_ip" default="0.0.0.0"/>
-  <xacro:arg name="script_command_port" default="50004"/>
-  <xacro:arg name="reverse_port" default="50001"/>
-  <xacro:arg name="script_sender_port" default="50002"/>
-  <xacro:arg name="trajectory_port" default="50003"/>
-  <!--   tool communication related parameters-->
-  <xacro:arg name="use_tool_communication" default="false" />
-  <xacro:arg name="tool_voltage" default="0" />
-  <xacro:arg name="tool_parity" default="0" />
-  <xacro:arg name="tool_baud_rate" default="115200" />
-  <xacro:arg name="tool_stop_bits" default="1" />
-  <xacro:arg name="tool_rx_idle_chars" default="1.5" />
-  <xacro:arg name="tool_tx_idle_chars" default="3.5" />
-  <xacro:arg name="tool_device_name" default="/tmp/ttyUR" />
-  <xacro:arg name="tool_tcp_port" default="54321" />
-    <!-- Simulation parameters -->
-  <xacro:arg name="use_mock_hardware" default="false" />
-  <xacro:arg name="mock_sensor_commands" default="false" />
-  <xacro:arg name="simulation_controllers" default="" />
-  <!-- initial position for simulations (Mock Hardware, Gazebo, Ignition) -->
-  <xacro:arg name="initial_positions_file" default="$(find ur_description)/config/initial_positions.yaml"/>
-  <!-- convert to property to use substitution in function -->
-  <xacro:property name="initial_positions_file" default="$(arg initial_positions_file)"/>
-  <!-- create link fixed to the "world" -->
-  <link name="world" />
-  <xacro:ur_robot
-    name="$(arg name)"
-    tf_prefix="$(arg tf_prefix)"
-    parent="world"
-    joint_limits_parameters_file="$(arg joint_limit_params)"
-    kinematics_parameters_file="$(arg kinematics_params)"
-    physical_parameters_file="$(arg physical_params)"
-    visual_parameters_file="$(arg visual_params)"
-    safety_limits="$(arg safety_limits)"
-    safety_pos_margin="$(arg safety_pos_margin)"
-    safety_k_position="$(arg safety_k_position)"
-    >
+   <!-- robot name parameter -->
+   <xacro:arg name="name" default="ur"/>
+   <!-- import main macro -->
+   <xacro:include filename="$(find ur_description)/urdf/ur_macro.xacro"/>
+   <!-- possible 'ur_type' values: ur3, ur3e, ur5, ur5e, ur7e, ur10, ur10e, ur12e, ur16e, ur15, ur20, ur30 -->
+   <!-- the default value should raise an error in case this was called without defining the type -->
+   <xacro:arg name="ur_type" default="ur5x"/>
+   <!-- parameters -->
+   <xacro:arg name="tf_prefix" default="" />
+   <xacro:arg name="joint_limit_params" default="$(find ur_description)/config/$(arg ur_type)/joint_limits.yaml"/>
+   <xacro:arg name="kinematics_params" default="$(find ur_description)/config/$(arg ur_type)/default_kinematics.yaml"/>
+   <xacro:arg name="physical_params" default="$(find ur_description)/config/$(arg ur_type)/physical_parameters.yaml"/>
+   <xacro:arg name="visual_params" default="$(find ur_description)/config/$(arg ur_type)/visual_parameters.yaml"/>
+   <xacro:arg name="transmission_hw_interface" default=""/>
+   <xacro:arg name="safety_limits" default="false"/>
+   <xacro:arg name="safety_pos_margin" default="0.15"/>
+   <xacro:arg name="safety_k_position" default="20"/>
+   <!-- ros2_control related parameters -->
+   <xacro:arg name="headless_mode" default="false" />
+   <xacro:arg name="robot_ip" default="0.0.0.0" />
+   <xacro:arg name="script_filename" default=""/>
+   <xacro:arg name="output_recipe_filename" default=""/>
+   <xacro:arg name="input_recipe_filename" default=""/>
+   <xacro:arg name="reverse_ip" default="0.0.0.0"/>
+   <xacro:arg name="script_command_port" default="50004"/>
+   <xacro:arg name="reverse_port" default="50001"/>
+   <xacro:arg name="script_sender_port" default="50002"/>
+   <xacro:arg name="trajectory_port" default="50003"/>
+   <!--   tool communication related parameters-->
+   <xacro:arg name="use_tool_communication" default="false" />
+   <xacro:arg name="tool_voltage" default="0" />
+   <xacro:arg name="tool_parity" default="0" />
+   <xacro:arg name="tool_baud_rate" default="115200" />
+   <xacro:arg name="tool_stop_bits" default="1" />
+   <xacro:arg name="tool_rx_idle_chars" default="1.5" />
+   <xacro:arg name="tool_tx_idle_chars" default="3.5" />
+   <xacro:arg name="tool_device_name" default="/tmp/ttyUR" />
+   <xacro:arg name="tool_tcp_port" default="54321" />
+     <!-- Simulation parameters -->
+   <xacro:arg name="use_fake_hardware" default="false" />
+   <xacro:arg name="fake_sensor_commands" default="false" />
+   <xacro:arg name="sim_gazebo" default="false" />
+   <xacro:arg name="sim_ignition" default="false" />
+   <xacro:arg name="simulation_controllers" default="" />
+   <!-- initial position for simulations (Fake Hardware, Gazebo, Ignition) -->
+   <xacro:arg name="initial_positions_file" default="$(find ur_description)/config/initial_positions.yaml"/>
+   <!-- convert to property to use substitution in function -->
+   <xacro:property name="initial_positions_file" default="$(arg initial_positions_file)"/>
+   <xacro:property name="is_sim_gazebo" value="$(arg sim_gazebo)"/>
+   <xacro:property name="is_sim_ignition" value="$(arg sim_ignition)"/>
+   <!-- create link fixed to the "world" -->
+   <link name="world" />
+   <xacro:if value="${is_sim_gazebo or is_sim_ignition}">
+     <link name="ground_plane">
+       <visual>
+         <origin rpy="0 0 0" xyz="0 0 0"/>
+         <geometry>
+           <box size="5 5 0"/>
+         </geometry>
+         <material name="ground_white">
+           <color rgba="1 1 1 0.5"/>
+         </material>
+       </visual>
+       <collision>
+         <origin rpy="0 0 0" xyz="0 0 0"/>
+         <geometry>
+           <box size="5 5 0"/>
+         </geometry>
+       </collision>
+     </link>
+     <joint name="ground_plane_joint" type="fixed">
+       <origin xyz="0 0 -0.01" rpy="0 0 0"/>
+       <parent link="world"/>
+       <child link="ground_plane"/>
+     </joint>
+   </xacro:if>
+   <!-- arm -->
+   <xacro:ur_robot
+     name="$(arg name)"
+     tf_prefix="$(arg tf_prefix)"
+     parent="world"
+     joint_limits_parameters_file="$(arg joint_limit_params)"
+     kinematics_parameters_file="$(arg kinematics_params)"
+     physical_parameters_file="$(arg physical_params)"
+     visual_parameters_file="$(arg visual_params)"
+     safety_limits="$(arg safety_limits)"
+     safety_pos_margin="$(arg safety_pos_margin)"
+     safety_k_position="$(arg safety_k_position)"
+     use_fake_hardware="$(arg use_fake_hardware)"
+     fake_sensor_commands="$(arg fake_sensor_commands)"
+     sim_gazebo="$(arg sim_gazebo)"
+     sim_ignition="$(arg sim_ignition)"
+     headless_mode="$(arg headless_mode)"
+     initial_positions="${xacro.load_yaml(initial_positions_file)}"
+     use_tool_communication="$(arg use_tool_communication)"
+     tool_voltage="$(arg tool_voltage)"
+     tool_parity="$(arg tool_parity)"
+     tool_baud_rate="$(arg tool_baud_rate)"
+     tool_stop_bits="$(arg tool_stop_bits)"
+     tool_rx_idle_chars="$(arg tool_rx_idle_chars)"
+     tool_tx_idle_chars="$(arg tool_tx_idle_chars)"
+     tool_device_name="$(arg tool_device_name)"
+     tool_tcp_port="$(arg tool_tcp_port)"
+     robot_ip="$(arg robot_ip)"
+     script_filename="$(arg script_filename)"
+     output_recipe_filename="$(arg output_recipe_filename)"
+     input_recipe_filename="$(arg input_recipe_filename)"
+     reverse_ip="$(arg reverse_ip)"
+     script_command_port="$(arg script_command_port)"
+     reverse_port="$(arg reverse_port)"
+     script_sender_port="$(arg script_sender_port)"
+     trajectory_port="$(arg trajectory_port)"
+     >
      <origin xyz="0 0 0" rpy="0 0 0" />          <!-- position robot in the world -->
-  </xacro:ur_robot>
-  <!-- ros2 control instance -->
-  <xacro:ur_ros2_control
-    name="$(arg name)"
-    tf_prefix="$(arg tf_prefix)"
-    kinematics_parameters_file="$(arg kinematics_params)"
-    transmission_hw_interface="$(arg transmission_hw_interface)"
-    use_mock_hardware="$(arg use_mock_hardware)"
-    mock_sensor_commands="$(arg mock_sensor_commands)"
-    headless_mode="$(arg headless_mode)"
-    initial_positions="${xacro.load_yaml(initial_positions_file)}"
-    use_tool_communication="$(arg use_tool_communication)"
-    tool_voltage="$(arg tool_voltage)"
-    tool_parity="$(arg tool_parity)"
-    tool_baud_rate="$(arg tool_baud_rate)"
-    tool_stop_bits="$(arg tool_stop_bits)"
-    tool_rx_idle_chars="$(arg tool_rx_idle_chars)"
-    tool_tx_idle_chars="$(arg tool_tx_idle_chars)"
-    tool_device_name="$(arg tool_device_name)"
-    tool_tcp_port="$(arg tool_tcp_port)"
-    robot_ip="$(arg robot_ip)"
-    script_filename="$(arg script_filename)"
-    output_recipe_filename="$(arg output_recipe_filename)"
-    input_recipe_filename="$(arg input_recipe_filename)"
-    reverse_ip="$(arg reverse_ip)"
-    script_command_port="$(arg script_command_port)"
-    reverse_port="$(arg reverse_port)"
-    script_sender_port="$(arg script_sender_port)"
-    trajectory_port="$(arg trajectory_port)"
-  />
+   </xacro:ur_robot>
+   <xacro:if value="$(arg sim_gazebo)">
+    <!-- Gazebo plugins -->
+    <gazebo reference="world">
+    </gazebo>
+    <gazebo>
+      <plugin filename="libgazebo_ros2_control.so" name="gazebo_ros2_control">
+        <parameters>$(arg simulation_controllers)</parameters>
+      </plugin>
+    </gazebo>
+  </xacro:if>
+  <xacro:if value="$(arg sim_ignition)">
+    <!-- Gazebo plugins -->
+    <gazebo reference="world">
+    </gazebo>
+    <gazebo>
+      <plugin filename="libign_ros2_control-system.so" name="ign_ros2_control::IgnitionROS2ControlPlugin">
+        <parameters>$(arg simulation_controllers)</parameters>
+        <controller_manager_node_name>$(arg tf_prefix)controller_manager</controller_manager_node_name>
+      </plugin>
+    </gazebo>
+  </xacro:if>
+  <!-- Import macros -->
+  <xacro:include filename="$(find robotiq_description)/urdf/robotiq_2f_85_macro.urdf.xacro" />
+  <xacro:robotiq_gripper name="RobotiqGripperHardwareInterface" prefix="" parent="tool0" use_fake_hardware="$(arg use_fake_hardware)" com_port="$(arg com_port)">
+      <origin xyz="0 0 0" rpy="0 0 0" />
+  </xacro:robotiq_gripper>
 </robot>

Commit message: update xacro

File: urdf/ur.urdf.xacro (robot description, xacro)
@@ -139,6 +139,24 @@
   <!-- Import macros -->
   <xacro:include filename="$(find robotiq_description)/urdf/robotiq_2f_85_macro.urdf.xacro" />
-  <xacro:robotiq_gripper name="RobotiqGripperHardwareInterface" prefix="" parent="tool0" use_fake_hardware="$(arg use_fake_hardware)" com_port="$(arg com_port)">
+  <link name="camera"/>
+    <joint name="camera_joint" type="fixed">
+        <origin xyz="0 0 0.005" rpy="0 0 0"/>
+        <parent link="tool0"/>
+        <child link="camera"/>
+    </joint>
+  <link name="force_sensor"/>
+    <joint name="force_sensor_joint" type="fixed">
+        <origin xyz="0 0 0.045" rpy="0 0 0"/>
+        <parent link="camera"/>
+        <child link="force_sensor"/>
+    </joint>
+  <xacro:robotiq_gripper name="RobotiqGripperHardwareInterface" prefix="" parent="force_sensor" use_fake_hardware="$(arg use_fake_hardware)" com_port="$(arg com_port)">
       <origin xyz="0 0 0" rpy="0 0 0" />
   </xacro:robotiq_gripper>
+  <link name="finger_center"/>
+    <joint name="finger_center_joint" type="fixed">
+        <origin xyz="0 0 0.20" rpy="0 0 0"/>
+        <parent link="tool0"/>
+        <child link="finger_center"/>
+    </joint>
 </robot>

File: urdf/ur_gripper.urdf.xacro (robot description, xacro)
@@ -101,3 +101,9 @@
         <origin xyz="0 0 0" rpy="0 0 0" />
     </xacro:robotiq_gripper>
+    <link name="finger_center"/>
+    <joint name="finger_center_joint" type="fixed">
+        <origin xyz="0 0 0.20" rpy="0 0 0"/>
+        <parent link="tool0"/>
+        <child link="finger_center"/>
+    </joint>
 </robot>

Commit message: adapt real hardware

File: urdf/ur.urdf.xacro (robot description, xacro)
@@ -139,22 +139,95 @@
   <!-- Import macros -->
   <xacro:include filename="$(find robotiq_description)/urdf/robotiq_2f_85_macro.urdf.xacro" />
-  <link name="camera"/>
+    <link name="realsense_camera">
+    <visual>
+        <origin rpy="-1.5707963267948966 0 0" xyz="0 0 -0.005"/>
+        <geometry>
+            <mesh filename="package://ur5_robot_gripper/meshes/realsense/visual/realsense.dae"/>
+        </geometry>
+    </visual>
+    <collision>
+        <origin rpy="1.5707963267948966 0 0" xyz="0 0 -0.005"/>
+        <geometry>
+            <mesh filename="package://ur5_robot_gripper/meshes/realsense/collision/realsense.stl"/>
+        </geometry>
+    </collision>
+    </link>
     <joint name="camera_joint" type="fixed">
         <origin xyz="0 0 0.005" rpy="0 0 0"/>
         <parent link="tool0"/>
-        <child link="camera"/>
-    </joint>
-  <link name="force_sensor"/>
-    <joint name="force_sensor_joint" type="fixed">
-        <origin xyz="0 0 0.045" rpy="0 0 0"/>
-        <parent link="camera"/>
-        <child link="force_sensor"/>
-    </joint>
-  <xacro:robotiq_gripper name="RobotiqGripperHardwareInterface" prefix="" parent="force_sensor" use_fake_hardware="$(arg use_fake_hardware)" com_port="$(arg com_port)">
+        <child link="realsense_camera"/>
+    </joint>
+    <!-- mount the fts to the robot -->
+    <joint name="ft300_fix" type="fixed">
+      <origin rpy="0 0 0" xyz="0 0 0"/>
+      <parent link="realsense_camera"/>
+      <child link="ft300_mounting_plate"/>
+    </joint>
+    <!-- Link representing the FT300 force-torque sensor -->
+    <link name="ft300_sensor">
+      <inertial>
+        <origin rpy="0 0 0" xyz="0 0 -0.017"/>
+        <mass value="0.300"/>
+        <inertia ixx="0.000262" ixy="0" ixz="1e-06" iyx="0" iyy="0.000265" iyz="1e-06" izx="-1e-06" izy="1e-06" izz="0.000219"/>
+      </inertial>
+      <visual>
+        <origin rpy="0 0 0" xyz="0 0 0"/>
+        <geometry>
+          <mesh filename="package://ur5_robot_gripper/meshes/ft300/visual/robotiq_ft300.STL"/>
+        </geometry>
+        <material name="Robotiq-Black">
+          <color rgba="0.2 0.2 0.2 1.0"/>
+        </material>
+      </visual>
+      <collision>
+        <origin rpy="0 0 0" xyz="0 0 0"/>
+        <geometry>
+          <mesh filename="package://ur5_robot_gripper/meshes/ft300/collision/robotiq_ft300.STL"/>
+        </geometry>
+      </collision>
+    </link>
+    <!-- Link representing the FT300 mounting plate -->
+    <link name="ft300_mounting_plate">
+      <visual>
+        <origin rpy="0 0 0" xyz="0 0 0"/>
+        <geometry>
+          <mesh filename="package://ur5_robot_gripper/meshes/ft300/visual/mountings/robotiq_ft300-G-062-COUPLING_G-50-4M6-1D6_20181119.STL"/>
+        </geometry>
+        <material name="Robotiq-Grey">
+          <color rgba="0.4 0.4 0.4 1.0"/>
+        </material>
+      </visual>
+      <collision>
+        <origin rpy="0 0 0" xyz="0 0 0"/>
+        <geometry>
+          <mesh filename="package://ur5_robot_gripper/meshes/ft300/collision/mountings/robotiq_ft300-G-062-COUPLING_G-50-4M6-1D6_20181119.STL"/>
+        </geometry>
+      </collision>
+    </link>
+    <!-- Connect force sensor with mounting/coupling plate -->
+    <joint name="ft300_mounting_plate" type="fixed">
+      <origin rpy="0 3.141592653589793 0" xyz="0 0 0.0415"/>
+      <parent link="ft300_mounting_plate"/>
+      <child link="ft300_sensor"/>
+    </joint>
+    <!-- FORCE REFERENCE FRAME _______________________________________________________________________________
+              As specified in the documentation:
+              - The Z axis passes through the center of the depression with positive direction in the tool direction.
+              - The X axis traces a symmetric line centered on the connector; the positive direction
+                  points the opposite way away from the connector.
+              - The Y axis uses the right hand thumb rule according to X-Z. -->
+    <joint name="measurment_joint" type="fixed">
+      <origin rpy="0 3.141592653589793 0" xyz="0 0 0"/>
+      <parent link="ft300_sensor"/>
+      <child link="robotiq_ft_frame_id"/>
+    </joint>
+    <link name="robotiq_ft_frame_id"/>
+  <xacro:robotiq_gripper name="RobotiqGripperHardwareInterface" prefix="" parent="robotiq_ft_frame_id" use_fake_hardware="$(arg use_fake_hardware)" com_port="$(arg com_port)">
       <origin xyz="0 0 0" rpy="0 0 0" />
   </xacro:robotiq_gripper>
+  <!-- change this together with the xacro file: ur_robotiq.urdf because moveit with use the urdf file to generate the ik solver -->
   <link name="finger_center"/>
     <joint name="finger_center_joint" type="fixed">
-        <origin xyz="0 0 0.20" rpy="0 0 0"/>
+        <origin xyz="0 0 0.208" rpy="0 0 0"/>
         <parent link="tool0"/>
         <child link="finger_center"/>

File: urdf/ur_robotiq.urdf (robot description, URDF)
Before this commit: robot ur5, 23 links, 22 joints
Joints:
- joint finger_center_joint: origin xyz=0 0 0.20 rpy=0 0 0 -> xyz=0 0 0.208 rpy=0 0 0

Commit message: fix wrong camera installation

File: urdf/ur.urdf.xacro (robot description, xacro)
@@ -147,5 +147,5 @@
     </visual>
     <collision>
-        <origin rpy="1.5707963267948966 0 0" xyz="0 0 -0.005"/>
+        <origin rpy="-1.5707963267948966 0 0" xyz="0 0 -0.005"/>
         <geometry>
             <mesh filename="package://ur5_robot_gripper/meshes/realsense/collision/realsense.stl"/>

Commit message: use correct urdf

File: urdf/ur.urdf.xacro (robot description, xacro)
@@ -229,6 +229,6 @@
   <link name="finger_center"/>
     <joint name="finger_center_joint" type="fixed">
-        <origin xyz="0 0 0.208" rpy="0 0 0"/>
-        <parent link="tool0"/>
+        <origin xyz="0 0 0.16" rpy="0 0 0"/>
+        <parent link="robotiq_ft_frame_id"/>
         <child link="finger_center"/>
     </joint>
