Commit message: add ros2 branch

File: urdf/robotiq_gripper/robotiq.xacro (robot description, xacro)
@@ -1,9 +1,8 @@
 <?xml version="1.0"?>
 <robot name="ur5_with_robotiq_2f_85" xmlns:xacro="http://www.ros.org/wiki/xacro">
-    <!-- Include UR5 xacro -->
-    <xacro:include filename="$(find ur5_robot_gripper)/urdf/ur5/ur5.xacro" />
     <!-- Include Robotiq 2F-85 xacro -->
     <xacro:include filename="$(find ur5_robot_gripper)/urdf/robotiq_gripper/robotiq_85_gripper.urdf.xacro" />
-    <xacro:robotiq_85_gripper prefix="" parent="tool0" >
+    <link name="world"/>
+    <xacro:robotiq_85_gripper prefix="" parent="world" >
     <origin xyz="0 0 0.004" rpy="0 ${-pi/2} ${pi/2}"/>
     </xacro:robotiq_85_gripper>
