Commit message: :wrench: add joint limits for curobo

File: meshes/ur5.urdf (robot description, URDF)
Before this commit: robot ur5, 21 links, 20 joints
Joints:
- joint wrist_2_joint: limit lower=-6.283185307179586 upper=6.283185307179586 effort=28.0 velocity=3.141592653589793 -> lower=-3.1415926535897931 upper=0.31415926535897931 effort=28.0 velocity=3.141592653589793

Commit message: remove joint limits for curobo js plan debugging

File: meshes/ur5.urdf (robot description, URDF)
Before this commit: robot ur5, 21 links, 20 joints
Joints:
- joint wrist_2_joint: limit lower=-3.1415926535897931 upper=0.31415926535897931 effort=28.0 velocity=3.141592653589793 -> lower=-3.1415926535897931 upper=3.1415926535897931 effort=28.0 velocity=3.141592653589793

Commit message: :bug: use 0.16 as finger center to tool0 position

File: meshes/ur5.urdf (robot description, URDF)
Before this commit: robot ur5, 21 links, 20 joints
Joints:
- joint tool0-finger_center: origin xyz=0 0 0.15 rpy=0 0 0 -> xyz=0 0 0.16 rpy=0 0 0
