Commit message: update robot models for isaac testing

File: meshes/ur5_gripper.urdf (robot description, URDF)
Before this commit: robot ur5, 12 links, 11 joints
Links:
- added link robotiq_85_base_link, mass 0.636951; collision mesh filename=robotiq/collision/robotiq_85_base_link.stl; visual mesh filename=robotiq/visual/robotiq_85_base_link.dae
- added link robotiq_85_left_finger_link, mass 0.027309; collision mesh filename=robotiq/collision/robotiq_85_finger_link.stl; visual mesh filename=robotiq/visual/robotiq_85_finger_link.dae
- added link robotiq_85_left_finger_tip_link, mass 0.019555; collision mesh filename=robotiq/collision/robotiq_85_finger_tip_link.stl; visual mesh filename=robotiq/visual/robotiq_85_finger_tip_link.dae
- added link robotiq_85_left_inner_knuckle_link, mass 0.029951; collision mesh filename=robotiq/collision/robotiq_85_inner_knuckle_link.stl; visual mesh filename=robotiq/visual/robotiq_85_inner_knuckle_link.dae
- added link robotiq_85_left_knuckle_link, mass 0.018491; collision mesh filename=robotiq/collision/robotiq_85_knuckle_link.stl; visual mesh filename=robotiq/visual/robotiq_85_knuckle_link.dae
- added link robotiq_85_right_finger_link, mass 0.027309; collision mesh filename=robotiq/collision/robotiq_85_finger_link.stl; visual mesh filename=robotiq/visual/robotiq_85_finger_link.dae
- added link robotiq_85_right_finger_tip_link, mass 0.019555; collision mesh filename=robotiq/collision/robotiq_85_finger_tip_link.stl; visual mesh filename=robotiq/visual/robotiq_85_finger_tip_link.dae
- added link robotiq_85_right_inner_knuckle_link, mass 0.029951; collision mesh filename=robotiq/collision/robotiq_85_inner_knuckle_link.stl; visual mesh filename=robotiq/visual/robotiq_85_inner_knuckle_link.dae
- added link robotiq_85_right_knuckle_link, mass 0.018491; collision mesh filename=robotiq/collision/robotiq_85_knuckle_link.stl; visual mesh filename=robotiq/visual/robotiq_85_knuckle_link.dae
Joints:
- added joint robotiq_85_base_joint: type fixed, parent tool0, child robotiq_85_base_link, origin xyz=0 0 0.004 rpy=0 -1.5707963267948966 1.5707963267948966
- added joint robotiq_85_left_finger_joint: type fixed, parent robotiq_85_left_knuckle_link, child robotiq_85_left_finger_link, origin xyz=-0.00408552455 -0.03148604435 0.0 rpy=0 0 0
- added joint robotiq_85_left_finger_tip_joint: type revolute, parent robotiq_85_left_inner_knuckle_link, child robotiq_85_left_finger_tip_link, origin xyz=0.04303959807 -0.03759940821 0.0 rpy=0.0 0.0 0.0, axis 0 0 1, limit lower=-3.14 upper=3.14 effort=0.1 velocity=100.0, mimic joint=robotiq_85_left_knuckle_joint multiplier=-1
- added joint robotiq_85_left_inner_knuckle_joint: type revolute, parent robotiq_85_base_link, child robotiq_85_left_inner_knuckle_link, origin xyz=0.06142 0.0127 0 rpy=3.141592653589793 0.0 0.0, axis 0 0 1, limit lower=0 upper=0.8757 effort=0.1 velocity=100.0, mimic joint=robotiq_85_left_knuckle_joint offset=0
- added joint robotiq_85_left_knuckle_joint: type revolute, parent robotiq_85_base_link, child robotiq_85_left_knuckle_link, origin xyz=0.05490451627 0.03060114443 0.0 rpy=3.141592653589793 0.0 0.0, axis 0 0 1, limit lower=0.0 upper=0.80285 effort=1000 velocity=0.5
- added joint robotiq_85_right_finger_joint: type fixed, parent robotiq_85_right_knuckle_link, child robotiq_85_right_finger_link, origin xyz=-0.00408552455 -0.03148604435 0.0 rpy=0 0 0
- added joint robotiq_85_right_finger_tip_joint: type revolute, parent robotiq_85_right_inner_knuckle_link, child robotiq_85_right_finger_tip_link, origin xyz=0.04303959807 -0.03759940821  0.0 rpy=0.0 0.0 0.0, axis 0 0 1, limit lower=-3.14 upper=3.14 effort=0.1 velocity=100.0, mimic joint=robotiq_85_left_knuckle_joint multiplier=-1
- added joint robotiq_85_right_inner_knuckle_joint: type revolute, parent robotiq_85_base_link, child robotiq_85_right_inner_knuckle_link, origin xyz=0.06142 -0.0127 0 rpy=0 0 0, axis 0 0 1, limit lower=0 upper=0.8757 effort=0.1 velocity=100.0, mimic joint=robotiq_85_left_knuckle_joint offset=0
- added joint robotiq_85_right_knuckle_joint: type revolute, parent robotiq_85_base_link, child robotiq_85_right_knuckle_link, origin xyz=0.05490451627 -0.03060114443 0.0 rpy=0.0 0.0 0.0, axis 0 0 1, limit lower=0 upper=0.80285 effort=1000 velocity=100.0, mimic joint=robotiq_85_left_knuckle_joint
